File: Wednesday/robotfrond/frond.withname.brd (EAGLE design)
At the start: 150 x 120 mm, 16 parts

Commit message: woll smoth approves of his new robot frond
git-svn-id: svn+ssh://bbfs-01.calit2.net/grw/Gordon/svn/trunk/Gadgets/Designs/CSE91Robots@22861 2cf53259-273a-af40-bda6-69d31023b8ec
Parts:
- moved DRVR_9_DRIVE 49.0 mm to (97.2, 94.5), turned to 270 degrees
- moved U$1_6_LED 29.8 mm to (82.3, 51.0)
- moved U$2_6_LED 29.3 mm to (72.2, 52.7)
- moved U$3_6_LED 19.9 mm to (82.7, 53.9)
- moved D1_1_BATTERY 17.7 mm to (93.9, 82.0), turned to 180 degrees
Connections:
- net A0_0_BRAIN: now also DRVR_9_DRIVE.AIN2; no longer DRVR_9_DRIVE.BIN2
- net A1_0_BRAIN: now also DRVR_9_DRIVE.BIN1
- net A2_0_BRAIN: now also DRVR_9_DRIVE.BIN2
- net D11_0_BRAIN: now also B1_7_BUTTON.P; no longer DRVR_9_DRIVE.AIN1
- net D12_0_BRAIN: now also DRVR_9_DRIVE.STBY; no longer DRVR_9_DRIVE.AIN2
- net D13_0_BRAIN: now also DRVR_9_DRIVE.AIN1; no longer DRVR_9_DRIVE.BIN1
- net D4_0_BRAIN: now also U1_4_BUZZER.+; no longer B1_7_BUTTON.P
- net D8_0_BRAIN: now also U$2_5_BUMP.A; no longer DRVR_9_DRIVE.STBY
- net RXD1_0_BRAIN: no longer U1_4_BUZZER.+
- net TXD1_0_BRAIN: no longer U$2_5_BUMP.A
Routing:
- net TXD1_0_BRAIN: track 188.4 -> 0.00 mm, vias 2 -> 0
- net D13_0_BRAIN: track 187.1 -> 41.0 mm, vias 2 -> 0
- net +5V_0_BRAIN: track 234.2 -> 333.4 mm, vias 2 -> 0
- net D8_0_BRAIN: track 43.1 -> 140.3 mm, vias 0 -> 2
- net A01_9_DRIVE: track 56.5 -> 140.8 mm, vias 0 -> 2
- net N$3_6_LED: track 120.1 -> 41.7 mm
- net D10_0_BRAIN: track 156.5 -> 78.4 mm
- net A02_9_DRIVE: track 50.4 -> 125.8 mm, vias 0 -> 2
- net D11_0_BRAIN: track 101.9 -> 29.3 mm, vias 2 -> 0
- net RXD1_0_BRAIN: track 70.3 -> 0.00 mm
- net A4_0_BRAIN: track 116.6 -> 182.2 mm
- net B02_9_DRIVE: track 51.7 -> 107.6 mm
- net B01_9_DRIVE: track 57.2 -> 111.8 mm
- net N$1_6_LED: track 84.4 -> 36.2 mm, vias 2 -> 0
- net A0_0_BRAIN: track 69.7 -> 28.8 mm
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