File: Wednesday/robotfrond/frond.withname.sch (EAGLE design)
At the start: 16 parts, among them U1_0_brain ADAFRUIT-PRO-TRINKET-5V-BOB, u1_2_caster CASTERADAFRUIT-3/4IN, u1_3_penholder PENHOLDER, u1_4_buzzer BUZZERPTH, u1_8_display_2 ADAFRUIT-1.2IN-8X8-LED-BACKPA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

Commit message: woll smoth approves of his new robot frond
git-svn-id: svn+ssh://bbfs-01.calit2.net/grw/Gordon/svn/trunk/Gadgets/Designs/CSE91Robots@22861 2cf53259-273a-af40-bda6-69d31023b8ec
Connections:
- net A0_0_brain: now also DRVR_9_drive.AIN2; no longer DRVR_9_drive.BIN2
- net A1_0_brain: now also DRVR_9_drive.BIN1
- net A2_0_brain: now also DRVR_9_drive.BIN2
- net D11_0_brain: now also B1_7_button.P; no longer DRVR_9_drive.AIN1
- net D12_0_brain: now also DRVR_9_drive.STBY; no longer DRVR_9_drive.AIN2
- net D13_0_brain: now also DRVR_9_drive.AIN1; no longer DRVR_9_drive.BIN1
- net D4_0_brain: now also u1_4_buzzer.1; no longer B1_7_button.P
- net D8_0_brain: now also U$2_5_bump.A; no longer DRVR_9_drive.STBY
- net RXD1_0_brain: no longer u1_4_buzzer.1
- net TXD1_0_brain: no longer U$2_5_bump.A
Changed lines of the file:
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@@
           <busses/>
           <nets>
+            <net name="D4_0_brain" class="0">
+              <segment>
+                <pinref part="u1_4_buzzer" gate="G$1" pin="1"/>
+              </segment>
+            </net>
             <net name="GND2_0_brain" class="0">
               <segment>
                 <pinref part="u1_4_buzzer" gate="G$1" pin="2"/>
-              </segment>
-            </net>
-            <net name="RXD1_0_brain" class="0">
-              <segment>
-                <pinref part="u1_4_buzzer" gate="G$1" pin="1"/>
               </segment>
             </net>
@@
           <busses/>
           <nets>
+            <net name="D8_0_brain" class="0">
+              <segment>
+                <pinref part="U$2_5_bump" gate="G$1" pin="A"/>
+                <wire x1="50.8" y1="53.34" x2="35.56" y2="53.34" width="0.1524" layer="91"/>
+                <label x="35.56" y="53.34" size="1.778" layer="95"/>
+              </segment>
+            </net>
             <net name="GND2_0_brain" class="0">
               <segment>
@@
               </segment>
             </net>
-            <net name="TXD1_0_brain" class="0">
-              <segment>
-                <pinref part="U$2_5_bump" gate="G$1" pin="A"/>
-                <wire x1="50.8" y1="53.34" x2="35.56" y2="53.34" width="0.1524" layer="91"/>
-                <label x="35.56" y="53.34" size="1.778" layer="95"/>
-              </segment>
-            </net>
           </nets>
         </sheet>
@@
           <busses/>
           <nets>
-            <net name="D4_0_brain" class="0">
+            <net name="D11_0_brain" class="0">
               <segment>
                 <pinref part="B1_7_button" gate="G$1" pin="P"/>
@@
             <net name="A0_0_brain" class="0">
               <segment>
+                <pinref part="DRVR_9_drive" gate="G$1" pin="AIN2"/>
+                <wire x1="-5.08" y1="17.78" x2="-10.16" y2="17.78" width="0.1524" layer="91"/>
+                <label x="-10.16" y="17.78" size="1.778" layer="95" rot="R180" xref="yes"/>
+              </segment>
+            </net>
+            <net name="A1_0_brain" class="0">
+              <segment>
+                <pinref part="DRVR_9_drive" gate="G$1" pin="BIN1"/>
+                <wire x1="-5.08" y1="10.16" x2="-10.16" y2="10.16" width="0.1524" layer="91"/>
+                <label x="-10.16" y="10.16" size="1.778" layer="95" rot="R180" xref="yes"/>
+              </segment>
+            </net>
+            <net name="A2_0_brain" class="0">
+              <segment>
                 <pinref part="DRVR_9_drive" gate="G$1" pin="BIN2"/>
                 <wire x1="-5.08" y1="7.62" x2="-10.16" y2="7.62" width="0.1524" layer="91"/>
@@
               </segment>
             </net>
-            <net name="D11_0_brain" class="0">
+            <net name="D12_0_brain" class="0">
+              <segment>
+                <pinref part="DRVR_9_drive" gate="G$1" pin="STBY"/>
+                <wire x1="-5.08" y1="12.7" x2="-10.16" y2="12.7" width="0.1524" layer="91"/>
+                <label x="-10.16" y="12.7" size="1.778" layer="95" rot="R180" xref="yes"/>
+              </segment>
+            </net>
+            <net name="D13_0_brain" class="0">
               <segment>
                 <pinref part="DRVR_9_drive" gate="G$1" pin="AIN1"/>
@@
               </segment>
             </net>
-            <net name="D12_0_brain" class="0">
-              <segment>
-                <pinref part="DRVR_9_drive" gate="G$1" pin="AIN2"/>
-                <wire x1="-5.08" y1="17.78" x2="-10.16" y2="17.78" width="0.1524" layer="91"/>
-                <label x="-10.16" y="17.78" size="1.778" layer="95" rot="R180" xref="yes"/>
-              </segment>
-            </net>
-            <net name="D13_0_brain" class="0">
-              <segment>
-                <pinref part="DRVR_9_drive" gate="G$1" pin="BIN1"/>
-                <wire x1="-5.08" y1="10.16" x2="-10.16" y2="10.16" width="0.1524" layer="91"/>
-                <label x="-10.16" y="10.16" size="1.778" layer="95" rot="R180" xref="yes"/>
-              </segment>
-            </net>
-            <net name="D8_0_brain" class="0">
-              <segment>
-                <pinref part="DRVR_9_drive" gate="G$1" pin="STBY"/>
-                <wire x1="-5.08" y1="12.7" x2="-10.16" y2="12.7" width="0.1524" layer="91"/>
-                <label x="-10.16" y="12.7" size="1.778" layer="95" rot="R180" xref="yes"/>
-              </segment>
-            </net>
