File: Wednesday/alexwilliams/jak.withname.brd (EAGLE design)
At the start: 150 x 100 mm, 23 parts

Commit message: Expanded drills because we have run out of 0.8mm
git-svn-id: svn+ssh://bbfs-01.calit2.net/grw/Gordon/svn/trunk/Gadgets/Designs/CSE91Robots@22863 2cf53259-273a-af40-bda6-69d31023b8ec
Parts:
- D1_1_BATTERY: value (none) -> 450mV
- U1_0_BRAIN: value (none) -> ADAFRUIT-PRO-TRINKET-5V-BOB
- U1_12_CASTER_2, U1_6_CASTER: value (none) -> CASTERADAFRUIT-3/4IN
- U1_2_DISPLAY: value (none) -> ADAFRUIT-1.2IN-8X8-LED-BACKPACK-BOB
- U1_3_BUZZER: value (none) -> BUZZERPTH
