File: Tuesday/dlj/BashKetchum.withname.brd (EAGLE design)
At the start: 130 x 90 mm, 15 parts

Commit message: Readme
git-svn-id: svn+ssh://bbfs-01.calit2.net/grw/Gordon/svn/trunk/Gadgets/Designs/CSE91Robots@22925 2cf53259-273a-af40-bda6-69d31023b8ec
Routing:
- net A1_0_BRAIN: track 21.9 -> 19.8 mm
- net GND2_0_BRAIN: track 290.4 -> 292.5 mm
