File: Wednesday/Joanna/PessimistPrime.withname.brd (EAGLE design)
At the start: 150 x 100 mm, 20 parts

Commit message: Readme
git-svn-id: svn+ssh://bbfs-01.calit2.net/grw/Gordon/svn/trunk/Gadgets/Designs/CSE91Robots@22925 2cf53259-273a-af40-bda6-69d31023b8ec
Parts:
- D1_1_BATTERY: value (none) -> 450mV
- DIST1_4_DISTANCESENSOR: value (none) -> ANALOG_DISTANCE_SENSOR
- U1_0_BRAIN: value (none) -> ADAFRUIT-PRO-TRINKET-5V-BOB
- U1_3_CASTER: value (none) -> CASTERADAFRUIT-3/4IN
- U1_5_DISPLAY_2: value (none) -> ADAFRUIT-1.2IN-8X8-LED-BACKPACK-BOB
Routing:
- net GND2_0_BRAIN: track 384.1 -> 387.8 mm
